Commit message: Added ball and socket joints to upper two wing components.

File: pigeon_flat_plate_with_tail/robots/pigeon_flat_plate_ballsocket.URDF (robot description, URDF)
Before this commit: robot pigeon_flat_plate_with_tail, 8 links, 7 joints
Links:
- added link left_elbow_pseudo_one
- added link left_elbow_pseudo_two
- added link left_shoulder_pseudo_one
- added link left_shoulder_pseudo_two
- added link left_wrist_pseudo_one
- added link left_wrist_pseudo_two
- added link right_elbow_pseudo_one
- added link right_elbow_pseudo_two
- added link right_shoulder_pseudo_one
- added link right_shoulder_pseudo_two
- added link right_wrist_pseudo_one
- added link right_wrist_pseudo_two
Joints:
- removed joint left_elbow
- removed joint left_shoulder
- removed joint left_wrist
- removed joint right_elbow
- removed joint right_shoulder
- removed joint right_wrist
- added joint left_elbow_pitch: type continuous, parent left_upper_wing, child left_elbow_pseudo_one, origin xyz=-0.0419980875771034 0 0 rpy=0 0 0, axis -1 0 0
- added joint left_elbow_roll: type continuous, parent left_elbow_pseudo_one, child left_elbow_pseudo_two, origin xyz=0 0 0 rpy=-1.5707963267949 0 0, axis 0 1 0
- added joint left_elbow_yaw: type continuous, parent left_elbow_pseudo_two, child left_mid_wing, origin xyz=0 0 0 rpy=1.5707963267949 0 0, axis 0 -1 0
- added joint left_shoulder_pitch: type continuous, parent torso, child left_shoulder_pseudo_one, origin xyz=-0.104961900175268 -0.00441963567052359 -0.0724066467540735 rpy=-1.5707963267949 0 0, axis -1 0 0
- added joint left_shoulder_roll: type continuous, parent left_shoulder_pseudo_one, child left_shoulder_pseudo_two, origin xyz=0 0 0 rpy=1.5707963267949 0 0, axis 0 1 0
- added joint left_shoulder_yaw: type continuous, parent left_shoulder_pseudo_two, child left_upper_wing, origin xyz=0 0 0 rpy=1.5707963267949 0 0, axis 0 -1 0
- added joint left_wrist_pitch: type continuous, parent left_wrist_pseudo_two, child left_hand_wing, origin xyz=0 0 0 rpy=1.5707963267949 0 0, axis 0 -1 0
- added joint left_wrist_roll: type continuous, parent left_wrist_pseudo_one, child left_wrist_pseudo_two, origin xyz=0 0 0 rpy=-1.5707963267949 0 0, axis 0 1 0
- added joint right_elbow_pitch: type continuous, parent right_upper_wing, child right_elbow_pseudo_one, origin xyz=-0.0419980875771034 0 0 rpy=0 0 0, axis -1 0 0
- added joint right_elbow_roll: type continuous, parent right_elbow_pseudo_one, child right_elbow_pseudo_two, origin xyz=0 0 0 rpy=-1.5707963267949 0 0, axis 0 1 0
- added joint right_elbow_yaw: type continuous, parent right_elbow_pseudo_two, child right_mid_wing, origin xyz=0 0 0 rpy=1.5707963267949 0 0, axis 0 -1 0
- added joint right_shoulder_pitch: type continuous, parent torso, child right_shoulder_pseudo_one, origin xyz=-0.02098331 -0.00441963567052359 -0.0724066467540735 rpy=1.5707963267949 0 3.14159265358979, axis -1 0 0
- added joint right_shoulder_roll: type continuous, parent right_shoulder_pseudo_one, child right_shoulder_pseudo_two, origin xyz=0 0 0 rpy=1.5707963267949 0 0, axis 0 1 0
- added joint right_shoulder_yaw: type continuous, parent right_shoulder_pseudo_two, child right_upper_wing, origin xyz=0 0 0 rpy=1.5707963267949 0 0, axis 0 -1 0
- added joint right_wrist_pitch: type continuous, parent right_wrist_pseudo_two, child right_hand_wing, origin xyz=0 0 0 rpy=1.5707963267949 0 0, axis 0 -1 0
- added joint right_wrist_roll: type continuous, parent right_wrist_pseudo_one, child right_wrist_pseudo_two, origin xyz=0 0 0 rpy=-1.5707963267949 0 0, axis 0 1 0
