Commit message: Continued work on Ball and Socket model. Added pigeon_2 model with accurate mass data from Harvard Lab

File: pigeon_flat_plate_with_ballsocket/robots/pigeon_flat_plate_with_ballsocket.URDF (robot description, URDF)
Before this commit: robot pigeon_flat_plate_with_ballsocket, 16 links, 15 joints
Links:
- link le_ghost_one: mass None -> 0
- link le_ghost_two: mass None -> 0
- link ls_ghost_one: mass None -> 0
- link ls_ghost_two: mass None -> 0
- link re_ghost_one: mass None -> 0
- link re_ghost_two: mass None -> 0
- link rs_ghost_one: mass None -> 0
- link rs_ghost_two: mass None -> 0
