Commit message: added test files with ghosts links to debug ball and socket issues, added Hooke Joint test file for same purpose, committed previously made changes to get everything up to date

File: pigeon_2/robots/pigeon_2.URDF (robot description, URDF)
Before this commit: robot pigeon_2, 16 links, 15 joints
Links:
- link le_ghost_one: mass None -> 0
- link le_ghost_two: mass None -> 0
- link ls_ghost_one: mass None -> 0
- link ls_ghost_two: mass None -> 0
- link re_ghost_one: mass None -> 0
- link re_ghost_two: mass None -> 0
- link rs_ghost_one: mass None -> 0.000000001
- link rs_ghost_two: mass None -> 0.000000001
