Commit message: improved pigeon_3 URDF

File: pigeon_4/robots/pigeon_4.URDF (robot description, URDF)
Before this commit: robot pigeon_3, 16 links, 15 joints
Links:
- removed link torso
- added link base_link, mass 0.266575552840038; visual mesh filename=../meshes/base_link.STL
- link left_hand_wing: mass 0.00605546068773544 -> 0.00605546079567198
- link left_mid_wing: mass 0.00923222139282928 -> 0.00923222139282933
- link left_upper_wing: mass 0.00478467934314603 -> 0.00478467934314601
- link right_hand_wing: mass 0.00605546068773547 -> 0.00605546079567203
- link right_mid_wing: mass 0.00923222139282928 -> 0.00923222139282937
Joints:
- joint left_elbow_pitch: axis -1 0 0 -> 1 0 0; origin xyz=0 0 0.005 rpy=0 0 0 -> xyz=0 0 0 rpy=0 0 0
- joint left_elbow_roll: origin xyz=-0.0419980875771034 0 0.0150543231592249 rpy=0 0 0 -> xyz=-0.0419980875771035 0 0.0150543231592251 rpy=0 0 0
- joint left_elbow_yaw: origin xyz=0 0 -0.005 rpy=0 0 0 -> xyz=0 0 0 rpy=0 0 0
- joint left_shoulder_pitch: axis -1 0 0 -> 1 0 0; origin xyz=0 0 0.005 rpy=0 0 0 -> xyz=0 0 0 rpy=0 0 0
- joint left_shoulder_roll: origin xyz=-0.042 -0.076979541052234 0 rpy=1.5707963267949 0 0 -> xyz=0.0769795410522341 -0.0419999999999997 0 rpy=1.5707963267949 6.12303176911189E-17 1.5707963267949; parent torso -> base_link
- joint left_shoulder_yaw: origin xyz=0 0 -0.005 rpy=0 0 0 -> xyz=0 0 0 rpy=0 0 0
- joint left_wrist_roll: axis 0 0 -1 -> 0 0 1; origin xyz=-0.0929625657844593 0 0 rpy=0 0 0 -> xyz=-0.238685400185835 -0.00200000000000001 0.125278459956794 rpy=0 0 0
- joint right_elbow_pitch: axis -1 0 0 -> 1 0 0; origin xyz=0 0 0.005 rpy=0 0 0 -> xyz=0 0 0 rpy=0 0 0
- joint right_elbow_roll: origin xyz=-0.0419980875771034 0 0.0100543231592249 rpy=0 0 3.14159265358979 -> xyz=0.238685400185836 -0.002 0.115278459956792 rpy=3.14159265358979 0 3.14159265358979
- joint right_elbow_yaw: axis 0 1 0 -> 0 -1 0; origin xyz=0 0 -0.005 rpy=0 0 -3.14159265358979 -> xyz=0 0 0 rpy=3.14159265358979 1.38777878078145E-15 3.14159265358979
- joint right_shoulder_pitch: axis -1 0 0 -> 1 0 0; origin xyz=0 0 0.005 rpy=0 0 0 -> xyz=0 0 0 rpy=0 0 0
- joint right_shoulder_roll: axis 0 0 -1 -> 0 0 1; origin xyz=0.042 -0.076979541052234 0 rpy=1.5707963267949 0 0 -> xyz=0.0869795410522339 0.0370000000000003 -0.00500000000000001 rpy=1.5707963267949 6.12303176911189E-17 1.5707963267949; parent torso -> base_link
- joint right_shoulder_yaw: axis 0 1 0 -> 0 -1 0; origin xyz=0 0 0 rpy=0 0 3.14159265358979 -> xyz=0.28568348776294 0.00700000000000001 0.130332783116016 rpy=3.14159265358979 0 3.14159265358979
- joint right_wrist_roll: axis 0 0 -1 -> 0 0 1; origin xyz=-0.0929625657844593 0 0 rpy=0 0 -4.16333634234434E-15 -> xyz=-0.0929625657844593 0 0 rpy=0 1.38777878078145E-15 0
- joint tail_joint: axis -1 0 0 -> 1 0 0; origin xyz=0 -0.229979541052234 0 rpy=1.5707963267949 0 0 -> xyz=0.229979541052234 0 0 rpy=1.5707963267949 6.12303176911189E-17 1.5707963267949; parent torso -> base_link
