Commit message: fixed minor descrepancies between the left and right sides of the pigeon so as to reduce sidways tumbling

File: pigeon_8/robots/pigeon_8.URDF (robot description, URDF)
Before this commit: robot pigeon_8, 16 links, 15 joints
Links:
- link right_hand_wing: mass 0.00605546079567203 -> 0.00605546079567201
- link right_mid_wing: mass 0.00923222139282932 -> 0.0092322213928293
Joints:
- joint left_wrist_roll: axis 0 0 -1 -> 0 0 1
- joint right_elbow_roll: origin xyz=-0.041998 0 0.010054 rpy=3.1416 1.5708 0 -> xyz=-0.041998 0 0.010054 rpy=3.141592653 1.5708 0
- joint right_elbow_yaw: origin xyz=0 0 0 rpy=3.1416 1.5708 0 -> xyz=0 0 0 rpy=3.141592653 1.5708 0
- joint right_shoulder_yaw: origin xyz=0 0 0 rpy=3.1416 1.5708 0 -> xyz=0 0 0 rpy=3.141592653 1.5708 0
- joint right_wrist_roll: axis 0 0 1 -> 0 0 -1; origin xyz=-0.092963 0 0 rpy=0 0 -3.3307E-14 -> xyz=-0.092963 0 0 rpy=0 0 -1.1102E-14
