Commit message: added pigeon_10, which now has a much cleaner URDF that works with the runFlapping simulation. It is now able to maintain a very short flight with a simple sinusoidal flapping motion

File: pigeon_10/robots/pigeon_10.URDF (robot description, URDF)
Before this commit: robot pigeon_8, 16 links, 15 joints
Links:
- link left_mid_wing: mass 0.0092322213928293 -> 0.00923222139282933
- link left_upper_wing: mass 0.00478467934314603 -> 0.00478467934314604
- link right_mid_wing: mass 0.0092322213928293 -> 0.00923222139282933
- link right_upper_wing: mass 0.00478467934314603 -> 0.00478467934314604
Joints:
- joint left_elbow_pitch: axis 0 0 1 -> 0 1 0; origin xyz=-0.005 0 0 rpy=0 0 0 -> xyz=0 0 0 rpy=0 0 0
- joint left_elbow_roll: axis 1 0 0 -> -1 0 0; origin xyz=-0.041998 0 -0.010054 rpy=3.141592653 -1.5708 0 -> xyz=-0.0150543231592249 0.0419980875771034 0 rpy=0 0 0
- joint left_elbow_yaw: axis 0 1 0 -> 0 0 -1; origin xyz=0 0 0 rpy=3.141592653 -1.5708 0 -> xyz=0 0 0 rpy=0 0 0
- joint left_shoulder_pitch: axis 0 0 1 -> 0 1 0; origin xyz=-0.005 0 0 rpy=0 0 0 -> xyz=0 0 0 rpy=0 0 0
- joint left_shoulder_roll: axis 1 0 0 -> -1 0 0; origin xyz=-0.07698 0.042 0 rpy=1.5708 0 0 -> xyz=-0.08198 0.042 0 rpy=0 0 0
- joint left_shoulder_yaw: axis 0 1 0 -> 0 0 -1; origin xyz=0 0 0 rpy=3.141592653 -1.5708 0 -> xyz=0 0 0 rpy=0 0 0
- joint left_wrist_roll: axis 0 0 1 -> -1 0 0; origin xyz=-0.092963 0 0 rpy=0 0 1.1102E-14 -> xyz=0.0190702213237429 0.0929625657844593 0 rpy=0 0 0
- joint right_elbow_pitch: axis 0 0 1 -> 0 1 0; origin xyz=-0.005 0 0 rpy=0 0 0 -> xyz=0 0 0 rpy=0 0 0
- joint right_elbow_roll: axis 1 0 0 -> -1 0 0; origin xyz=-0.041998 0 0.010054 rpy=3.141592653 1.5708 0 -> xyz=-0.0150543231592249 0.0419980875771034 0 rpy=0 0 0
- joint right_elbow_yaw: axis 0 -1 0 -> 0 0 -1; origin xyz=0 0 0 rpy=3.141592653 1.5708 0 -> xyz=0 0 0 rpy=0 0 0
- joint right_shoulder_pitch: axis 0 0 1 -> 0 1 0; origin xyz=-0.005 0 0 rpy=0 0 0 -> xyz=0 0 0 rpy=0 0 0
- joint right_shoulder_roll: axis 1 0 0 -> -1 0 0; origin xyz=-0.07698 -0.042 0 rpy=1.5708 0 0 -> xyz=-0.081979541052234 -0.042 0 rpy=3.14159265358979 0 0
- joint right_shoulder_yaw: axis 0 -1 0 -> 0 0 -1; origin xyz=0 0 0 rpy=3.141592653 1.5708 0 -> xyz=0 0 0 rpy=0 0 0
- joint right_wrist_roll: axis 0 0 -1 -> -1 0 0; origin xyz=-0.092963 0 0 rpy=0 0 -1.1102E-14 -> xyz=0.0190702213237429 0.0929625657844593 0 rpy=0 0 0
- joint tail_joint: axis -1 0 0 -> 0 1 0; origin xyz=-0.22998 0 0 rpy=-1.5708 -6.123E-17 -1.5708 -> xyz=-0.25849 0 0 rpy=0 0 0

Commit message: added runDihedral, which simply puts the wings in a 30 degree dihedral and launches the bird forwards. This showed two important things, first that we can get the simulation to run longer than 1 or 2 seconds, and second that even after remaining stable for a long flight, it is still prone to veering off to the side randomly

File: pigeon_10/robots/pigeon_10.URDF (robot description, URDF)
Before this commit: robot pigeon_10, 16 links, 15 joints
Joints:
- joint right_shoulder_roll: origin xyz=-0.081979541052234 -0.042 0 rpy=3.14159265358979 0 0 -> xyz=-0.08198 -0.042 0 rpy=3.14159265358979 0 0
