Commit message: Pigeon 12 is now fully working with new dimensions, and the findTrim function works with it (I modified the dimensions of the arrays to make them match)

File: pigeon_11/robots/pigeon_11.URDF (robot description, URDF)
Before this commit: robot pigeon_11, 17 links, 16 joints
Links:
- link left_hand_wing: geometry visual mesh filename=../meshes/left_hand_wing.STL
- link left_mid_wing: geometry visual mesh filename=../meshes/left_mid_wing.STL
- link left_shoulder_pitch_ghost: mass 6.4E-11 -> 0; geometry 
- link left_shoulder_roll_ghost: mass 6.4E-11 -> 0; geometry 
- link left_upper_wing: geometry visual mesh filename=../meshes/left_upper_wing.STL
- link left_wrist_pitch_ghost: mass 6.4E-11 -> 0; geometry 
- link left_wrist_roll_ghost: mass 6.4E-11 -> 0; geometry 
- link right_hand_wing: geometry visual mesh filename=../meshes/right_hand_wing.STL
- link right_mid_wing: geometry visual mesh filename=../meshes/right_mid_wing.STL
- link right_shoulder_pitch_ghost: mass 6.4E-11 -> 0; geometry 
- link right_shoulder_roll_ghost: mass 6.4E-11 -> 0; geometry 
- link right_upper_wing: geometry visual mesh filename=../meshes/right_upper_wing.STL
- link right_wrist_pitch_ghost: mass 6.4E-11 -> 0; geometry 
- link right_wrist_roll_ghost: mass 6.4E-11 -> 0; geometry 
- link tail: geometry visual mesh filename=../meshes/tail.STL
- link tail_pitch_ghost: mass 6.4E-11 -> 0; geometry 
- link torso: geometry visual mesh filename=../meshes/torso.STL

File: pigeon_12/robots/pigeon_12.URDF (robot description, URDF)
Before this commit: robot pigeon_12, 17 links, 16 joints
Links:
- link left_hand_wing: geometry visual mesh filename=../meshes/left_hand_wing.STL
- link left_mid_wing: geometry visual mesh filename=../meshes/left_mid_wing.STL
- link left_shoulder_pitch_ghost: mass 6.4E-11 -> 0; geometry 
- link left_shoulder_roll_ghost: mass 6.4E-11 -> 0; geometry 
- link left_upper_wing: geometry visual mesh filename=../meshes/left_upper_wing.STL
- link left_wrist_pitch_ghost: mass 6.4E-11 -> 0; geometry 
- link left_wrist_roll_ghost: mass 6.4E-11 -> 0; geometry 
- link right_hand_wing: geometry visual mesh filename=../meshes/right_hand_wing.STL
- link right_mid_wing: geometry visual mesh filename=../meshes/right_mid_wing.STL
- link right_shoulder_pitch_ghost: mass 6.4E-11 -> 0; geometry 
- link right_shoulder_roll_ghost: mass 6.4E-11 -> 0; geometry 
- link right_upper_wing: geometry visual mesh filename=../meshes/right_upper_wing.STL
- link right_wrist_pitch_ghost: mass 6.4E-11 -> 0; geometry 
- link right_wrist_roll_ghost: mass 6.4E-11 -> 0; geometry 
- link tail: geometry visual mesh filename=../meshes/tail.STL
- link tail_pitch_ghost: mass 6.4E-11 -> 0; geometry 
- link torso: geometry visual mesh filename=../meshes/torso.STL
Joints:
- joint right_elbow_yaw: axis 0 0 -0.999999999999914 -> 0 0 -1; origin xyz=-0.0249799919935937 -0.0350000000000001 0 rpy=-4.7636921195345E-17 -1.86542065973815E-17 3.21998553575834E-14 -> xyz=-0.0249799919935937 -0.0350000000000001 0 rpy=0 0 0
- joint right_shoulder_pitch: axis 0 -0.999999999999989 0 -> 0 -1 0; origin xyz=0 0 0 rpy=2.0291111002841E-17 2.74327909829207E-07 1.79851477442537E-15 -> xyz=0 0 0 rpy=0 0 0
- joint right_shoulder_roll: origin xyz=-0.08 -0.02235 -0.0185680248036409 rpy=-1.05554753939627E-07 0 0 -> xyz=-0.08 -0.02235 -0.0185680248036409 rpy=0 0 0
- joint right_shoulder_yaw: axis 0.999999999999925 0 0 -> 0 0 1; origin xyz=0 0 0 rpy=1.40686878583019E-18 -3.10627098790649E-17 -2.97269970499519E-14 -> xyz=0 0 0 rpy=0 0 0
- joint right_wrist_pitch: origin xyz=0 0 0 rpy=0 -2.74327909765118E-07 0 -> xyz=0 0 0 rpy=0 0 0
- joint right_wrist_roll: axis -0.999999999999925 0 0 -> -1 0 0; origin xyz=0.0519142912418186 -0.034999999999993 0 rpy=1.05554753965563E-07 -1.43731962028398E-17 2.46852419319722E-14 -> xyz=0.0519142912418186 -0.034999999999993 0 rpy=0 0 0
