Commit message: Still in the middle of a lot of things, namely texturing the models to work with the new visualizer, but I'm just passing along the current status of things

File: old_versions/pigeon_15/robots/pigeon_15.URDF (robot description, URDF)
Before this commit: robot pigeon_16, 29 links, 28 joints
Links:
- link left_fingers: mass 0.000401251982836981 -> 0; geometry visual mesh filename=../meshes/left_fingers.STL
- link left_hand_wing: mass 0.00775959953779963 -> 0.00775959953779964; geometry visual mesh filename=../meshes/left_hand_wing.STL
- link left_lower_leg: mass 0.000510246738865067 -> 0; geometry visual mesh filename=../meshes/left_lower_leg.STL
- link left_mid_leg: mass 0.00256764664162857 -> 0; geometry visual mesh filename=../meshes/left_mid_leg.STL
- link left_mid_wing: geometry visual mesh filename=../meshes/left_mid_wing.STL
- link left_thumb: mass 9.61830981744704E-05 -> 0; geometry visual mesh filename=../meshes/left_thumb.STL
- link left_upper_leg: mass 0.00426407166179982 -> 0; geometry visual mesh filename=../meshes/left_upper_leg.STL
- link left_upper_wing: mass 0.00612600003399721 -> 0.0061260000339972; geometry visual mesh filename=../meshes/left_upper_wing.STL
- link right_fingers: mass 0.000401251982836982 -> 0; geometry visual mesh filename=../meshes/right_fingers.STL
- link right_hand_wing: geometry visual mesh filename=../meshes/right_hand_wing.STL
- link right_lower_leg: mass 0.000510246738865067 -> 0; geometry visual mesh filename=../meshes/right_lower_leg.STL
- link right_mid_leg: mass 0.00256764664162857 -> 0; geometry visual mesh filename=../meshes/right_mid_leg.STL
- link right_mid_wing: geometry visual mesh filename=../meshes/right_mid_wing.STL
- link right_thumb: mass 9.61830981744704E-05 -> 0; geometry visual mesh filename=../meshes/right_thumb.STL
- link right_upper_leg: mass 0.00426407166179982 -> 0; geometry visual mesh filename=../meshes/right_upper_leg.STL
- link right_upper_wing: geometry visual mesh filename=../meshes/right_upper_wing.STL
- link tail: mass 0.00272207360126705 -> 0.0036249709593909; geometry visual mesh filename=../meshes/tail.STL
- link torso: geometry visual mesh filename=../meshes/torso.STL
Joints:
- joint left_elbow_yaw: origin xyz=-0.0249799919935936 -0.035 0 rpy=0 0 0 -> xyz=-0.0249799919935938 -0.0350000000000007 0 rpy=0 0 0
- joint left_shoulder_roll: origin xyz=-0.08 0.0223499999999987 -0.0185680248036425 rpy=0 0 0 -> xyz=-0.08 0.0223499999999991 -0.018568024803642 rpy=0 0 0
- joint right_elbow_yaw: axis 0 0 -0.999999999999914 -> 0 0 -1; origin xyz=-0.0249799919935937 -0.0350000000000001 0 rpy=-4.7636921195345E-17 -1.86542065973815E-17 3.21998553575834E-14 -> xyz=-0.0249799919935937 -0.0350000000000001 0 rpy=0 0 0
- joint right_shoulder_pitch: axis 0 -0.999999999999989 0 -> 0 -1 0; origin xyz=0 0 0 rpy=2.0291111002841E-17 2.74327909829207E-07 1.79851477442537E-15 -> xyz=0 0 0 rpy=0 0 0
- joint right_shoulder_roll: origin xyz=-0.08 -0.02235 -0.0185680248036409 rpy=-1.05554753939627E-07 0 0 -> xyz=-0.08 -0.02235 -0.0185680248036409 rpy=0 0 0
- joint right_shoulder_yaw: axis 0 0 -1 -> 0 0 1; origin xyz=0 0 0 rpy=1.40686878583019E-18 -3.10627098790649E-17 -2.97269970499519E-14 -> xyz=0 0 0 rpy=0 0 0
- joint right_wrist_pitch: origin xyz=0 0 0 rpy=0 -2.74327909765118E-07 0 -> xyz=0 0 0 rpy=0 0 0
- joint right_wrist_roll: axis -0.999999999999925 0 0 -> -1 0 0; origin xyz=0.0519142912418186 -0.034999999999993 0 rpy=1.05554753965563E-07 -1.43731962028398E-17 2.46852419319722E-14 -> xyz=0.0519142912418186 -0.034999999999993 0 rpy=0 0 0

File: pigeon_16/robots/pigeon_16_no_texture.URDF (robot description, URDF)
Before this commit: robot pigeon_16, 29 links, 28 joints
Links:
- link left_fingers: geometry visual mesh filename=../meshes/left_fingers.STL
- link left_hand_wing: geometry visual mesh filename=../meshes/left_hand_wing.STL
- link left_lower_leg: geometry visual mesh filename=../meshes/left_lower_leg.STL
- link left_mid_leg: geometry visual mesh filename=../meshes/left_mid_leg.STL
- link left_mid_wing: geometry visual mesh filename=../meshes/left_mid_wing.STL
- link left_thumb: geometry visual mesh filename=../meshes/left_thumb.STL
- link left_upper_leg: geometry visual mesh filename=../meshes/left_upper_leg.STL
- link left_upper_wing: geometry visual mesh filename=../meshes/left_upper_wing.STL
- link right_fingers: geometry visual mesh filename=../meshes/right_fingers.STL
- link right_hand_wing: geometry visual mesh filename=../meshes/right_hand_wing.STL
- link right_lower_leg: geometry visual mesh filename=../meshes/right_lower_leg.STL
- link right_mid_leg: geometry visual mesh filename=../meshes/right_mid_leg.STL
- link right_mid_wing: geometry visual mesh filename=../meshes/right_mid_wing.STL
- link right_thumb: geometry visual mesh filename=../meshes/right_thumb.STL
- link right_upper_leg: geometry visual mesh filename=../meshes/right_upper_leg.STL
- link right_upper_wing: geometry visual mesh filename=../meshes/right_upper_wing.STL
- link tail: geometry visual mesh filename=../meshes/tail.STL
- link torso: geometry visual mesh filename=../meshes/torso.STL
