Commit message: made compatible with old viewer

File: pigeon_17/urdf/pigeon_17.URDF (robot description, URDF)
Before this commit: robot pigeon_16, 29 links, 28 joints
Links:
- link left_fingers: geometry visual mesh filename=../meshes/fingers_texture.STL
- link left_hand_wing: geometry visual mesh filename=../meshes/left_hand_wing_texture.STL
- link left_lower_leg: geometry visual mesh filename=../meshes/lower_leg_texture.STL
- link left_mid_leg: geometry visual mesh filename=../meshes/mid_leg_texture.STL
- link left_mid_wing: geometry visual mesh filename=../meshes/left_mid_wing_texture.STL
- link left_thumb: geometry visual mesh filename=../meshes/thumb_texture.STL
- link left_upper_leg: geometry visual mesh filename=../meshes/upper_leg_texture.STL
- link left_upper_wing: geometry visual mesh filename=../meshes/left_upper_wing_texture.STL
- link right_fingers: geometry visual mesh filename=../meshes/fingers_texture.STL
- link right_hand_wing: geometry visual mesh filename=../meshes/left_hand_wing_texture.STL
- link right_lower_leg: geometry visual mesh filename=../meshes/lower_leg_texture.STL
- link right_mid_leg: geometry visual mesh filename=../meshes/mid_leg_texture.STL
- link right_mid_wing: geometry visual mesh filename=../meshes/left_mid_wing_texture.STL
- link right_thumb: geometry visual mesh filename=../meshes/thumb_texture.STL
- link right_upper_leg: geometry visual mesh filename=../meshes/upper_leg_texture.STL
- link right_upper_wing: geometry visual mesh filename=../meshes/left_upper_wing_texture.STL
- link tail: geometry visual mesh filename=../meshes/tail_texture.STL
- link torso: geometry visual mesh filename=../meshes/torso_texture.STL

Commit message: minor URDF fix, added animation script and video of said animation

File: pigeon_17/urdf/pigeon_17.URDF (robot description, URDF)
Before this commit: robot pigeon_16, 29 links, 28 joints
Joints:
- joint right_shoulder_yaw: axis 0.999999999999925 0 0 -> 0 0 -1

Commit message: updated URDF to include tail roll joint

File: pigeon_17/urdf/pigeon_17.URDF (robot description, URDF)
Before this commit: robot pigeon_16, 29 links, 28 joints
Links:
- added link tail_roll_ghost, mass 0
Joints:
- added joint tail_roll: type continuous, parent torso, child tail_roll_ghost, origin xyz=-0.21 0 -0.0185680248036409 rpy=0 0 0, axis -1 0 0
- joint tail_pitch: origin xyz=-0.21 0 -0.0185680248036409 rpy=0 0 0 -> xyz=0 0 0 rpy=0 0 0; parent torso -> tail_roll_ghost

Commit message: continuing work on findTrim

File: pigeon_17/urdf/pigeon_17.URDF (robot description, URDF)
Before this commit: robot pigeon_16, 30 links, 29 joints
Joints:
- joint right_elbow_yaw: axis 0 0 -0.999999999999914 -> 0 0 -1
- joint right_shoulder_pitch: axis 0 -0.999999999999989 0 -> 0 -1 0
- joint right_wrist_roll: axis -0.999999999999925 0 0 -> -1 0 0
